File: ECAD/MainBoardDifferential2026/MainBoardDifferential2026.kicad_pcb (KiCad board)
At the start: 2 copper layers, 58 x 105 mm, 58 parts, among them J1 NeoPixel, J100 Steppers, J12 Lidar LD06, J16 XT30, J2 XT60, J20 BAU, J22 BAU, J23 Conn_01x02, J24 External tools, J25 Conn_01x02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

Commit message: silkscreen
Parts:
- added G***: LOGO, LOGO, F.Cu at (162.0, 82.0)
- added G***: LOGO, LOGO, F.Cu at (184.5, 112.2)
- added G***: LOGO, LOGO, F.Cu at (157.5, 137.5)
- added G***: LOGO, LOGO, F.Cu at (185.5, 129.5)
- added G***: LOGO, LOGO, F.Cu at (146.9, 53.5)
- added G***: LOGO, LOGO, F.Cu at (163.8, 69.2)
- added G***: LOGO, LOGO, F.Cu at (175.2, 112.2)
- added G***: LOGO, LOGO, F.Cu at (162.0, 68.0)
- added G***: LOGO, LOGO, F.Cu at (145.1, 145.0)
- added G***: LOGO, LOGO, F.Cu at (183.0, 141.7)
- added G***: LOGO, LOGO, B.Cu at (141.4, 81.2)
- added G***: LOGO, LOGO, F.Cu at (138.5, 92.0)
- added G***: LOGO, LOGO, B.Cu at (174.8, 59.5)
- added G***: LOGO, LOGO, B.Cu at (165.5, 50.2)
- added G***: LOGO, LOGO, B.Cu at (149.0, 81.2)
- added G***: LOGO, LOGO, B.Cu at (191.5, 72.2)
- added G***: LOGO, LOGO, F.Cu at (153.0, 92.0)
- added G***: LOGO, LOGO, F.Cu at (145.5, 92.0)
- added G***: LOGO, LOGO, F.Cu at (139.3, 46.5)
- added G***: LOGO, LOGO, F.Cu at (164.2, 110.6)
- added G***: LOGO, LOGO, F.Cu at (163.2, 89.5)
- added G***: LOGO, LOGO, F.Cu at (160.0, 92.0)
- added G***: LOGO, LOGO, F.Cu at (150.4, 123.0)
- added kibuzzard-6493F09E: G***, kibuzzard-6493F09E, F.Cu at (175.0, 74.2)
- added kibuzzard-6493F0A8: G***, kibuzzard-6493F0A8, F.Cu at (175.0, 81.2)
- added kibuzzard-64944345: G***, kibuzzard-64944345, F.Cu at (156.6, 98.8)
- added kibuzzard-64944398: G***, kibuzzard-64944398, F.Cu at (141.7, 98.8)
- added kibuzzard-670C3331: G***, kibuzzard-670C3331, F.Cu at (142.4, 134.1)
- added kibuzzard-670C3331: G***, kibuzzard-670C3331, B.Cu at (147.7, 129.5)
- added kibuzzard-670C3352: G***, kibuzzard-670C3352, F.Cu at (158.0, 121.0)
- added kibuzzard-670C3352: G***, kibuzzard-670C3352, F.Cu at (171.2, 114.3)
- added kibuzzard-670C3352: G***, kibuzzard-670C3352, B.Cu at (147.7, 127.0)
- added kibuzzard-670C3359: G***, kibuzzard-670C3359, F.Cu at (175.2, 101.3)
- added kibuzzard-670C3359: G***, kibuzzard-670C3359, F.Cu at (163.8, 104.6)
- added kibuzzard-670C3359: G***, kibuzzard-670C3359, F.Cu at (186.8, 101.4)
- added kibuzzard-670C3359: G***, kibuzzard-670C3359, B.Cu at (147.7, 124.5)
- added kibuzzard-670C3379: G***, kibuzzard-670C3379, B.Cu at (147.8, 121.9)
- added kibuzzard-670C3380: G***, kibuzzard-670C3380, B.Cu at (147.7, 119.5)
- added kibuzzard-670C34D3: G***, kibuzzard-670C34D3, B.Cu at (140.5, 83.8)
- added kibuzzard-670C34D3: G***, kibuzzard-670C34D3, B.Cu at (174.6, 54.4)
- added kibuzzard-670C34F5: G***, kibuzzard-670C34F5, B.Cu at (174.4, 64.6)
- added kibuzzard-670C3554: G***, kibuzzard-670C3554, B.Cu at (181.5, 66.4)
- added kibuzzard-670C355C: G***, kibuzzard-670C355C, B.Cu at (181.9, 64.1)
- added kibuzzard-670C3560: G***, kibuzzard-670C3560, B.Cu at (181.6, 59.5)
- added kibuzzard-670C3565: G***, kibuzzard-670C3565, B.Cu at (181.5, 55.0)
- added kibuzzard-670C356A: G***, kibuzzard-670C356A, B.Cu at (181.7, 52.2)
- added kibuzzard-670C3571: G***, kibuzzard-670C3571, B.Cu at (174.1, 56.9)
- added kibuzzard-670C3577: G***, kibuzzard-670C3577, B.Cu at (173.9, 62.0)
- added kibuzzard-670C3646: G***, kibuzzard-670C3646, B.Cu at (140.6, 86.4)
- added kibuzzard-670C364B: G***, kibuzzard-670C364B, B.Cu at (140.5, 88.9)
- added kibuzzard-670C3872: G***, kibuzzard-670C3872, F.Cu at (167.8, 55.0)
- added kibuzzard-670C38FC: G***, kibuzzard-670C38FC, F.Cu at (156.0, 86.5)
- added kibuzzard-670C3904: G***, kibuzzard-670C3904, F.Cu at (156.0, 89.0)
Other:
- board text added: "BAU"
- board text added: "Barbatronic"
- board text added: "Karibous 2026"
- board text added: "MainBoard Differential Bot"
- board text added: "Même connecteurs MAIS tensions différentes"
- board text added: "Produced by Aisler"
